File: SBC6309Rom.kicad_sch (KiCad schematic)
At the start: 10 parts, among them J1 Address, J2 Device, J3 Clock, J4 Power, J5 Data, J6 Address select, U1 28C256, U6 GAL16V8

Commit message: fix rom footprint
Parts:
- U1: footprint Package_LCC:PLCC-28_THT-Socket -> Package_LCC:PLCC-32_THT-Socket; symbol Memory_EEPROM:28C256 -> Library:28C256
Connections:
- net +5V: now also U1.31 (~{WE}), U1.32 (VCC); no longer U1.27 (~{WE}), U1.28 (VCC)
- net A0: now also U1.11 (A0); no longer U1.10 (A0)
- net A1: now also U1.10 (A1); no longer U1.9 (A1)
- net A10: now also U1.24 (A10); no longer U1.21 (A10)
- net A11: now also U1.27 (A11); no longer U1.23 (A11)
- net A12: now also U1.3 (A12); no longer U1.2 (A12)
- net A2: now also U1.9 (A2); no longer U1.8 (A2)
- net A3: now also U1.8 (A3); no longer U1.7 (A3)
- net A4: now also U1.7 (A4); no longer U1.6 (A4)
- net A5: now also U1.6 (A5); no longer U1.5 (A5)
- net A6: now also U1.5 (A6); no longer U1.4 (A6)
- net A7: now also U1.4 (A7); no longer U1.3 (A7)
- net A8: now also U1.29 (A8); no longer U1.25 (A8)
- net A9: now also U1.28 (A9); no longer U1.24 (A9)
- net D0: now also U1.13 (D0); no longer U1.11 (D0)
- net D1: now also U1.14 (D1); no longer U1.12 (D1)
- net D2: now also U1.15 (D2); no longer U1.13 (D2)
- net D3: now also U1.18 (D3); no longer U1.15 (D3)
- net D4: now also U1.19 (D4); no longer U1.16 (D4)
- net D5: now also U1.20 (D5); no longer U1.17 (D5)
- net D6: now also U1.21 (D6); no longer U1.18 (D6)
- net D7: now also U1.22 (D7); no longer U1.19 (D7)
- net GND: now also U1.16 (GND); no longer U1.14 (GND)
- net ~{CS}: now also U1.23 (~{CS}); no longer U1.20 (~{CS})
- net ~{OE}: now also U1.25 (~{OE}); no longer U1.22 (~{OE})
- net at U1.26 (NC): no longer J6.4 (Pin_4)
- net at U1.1 (DC): no longer J6.6 (Pin_6)
- new net A13page: J6.4 (Pin_4), U1.30 (A13)
- new net A14page: J6.6 (Pin_6), U1.2 (A14)
Changed lines of the file:
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@@
+		)
+	)
+	(label "A13page"
+		(at 121.92 63.5 0)
+		(effects
+			(font
+				(size 1.27 1.27)
+			)
+			(justify left bottom)
 		)
 	)
@@
 	(label "D1"
 		(at 36.83 158.75 0)
+		(effects
+			(font
+				(size 1.27 1.27)
+			)
+			(justify left bottom)
+		)
+	)
+	(label "A14page"
+		(at 121.92 66.04 0)
 		(effects
 			(font
@@
 	)
 	(symbol
-		(lib_id "Memory_EEPROM:28C256")
+		(lib_id "Library:28C256")
 		(at 140.97 53.34 0)
 		(unit 1)
@@
 			)
 		)
-		(property "Footprint" "Package_LCC:PLCC-28_THT-Socket"
+		(property "Footprint" "Package_LCC:PLCC-32_THT-Socket"
 			(at 140.97 53.34 0)
 			(effects
@@
 			)
 		)
-		(property "Description" "Paged Parallel EEPROM 256Kb (32K x 8), DIP-28/SOIC-28"
+		(property "Description" "Paged Parallel EEPROM 256Kb (32K x 8), PLCC-32"
 			(at 140.97 53.34 0)
 			(effects
@@
 		(pin "19"
 		)
+		(pin "31"
+		)
+		(pin "29"
+		)
+		(pin "32"
+		)
+		(pin "30"
+		)
 		(instances
